Commit message: feat: optional suspension in sac_description; localization for 1 m GNSS
- sac_description: suspension:=true puts each wheel on a prismatic joint with a
  damper (1.4 Hz ride frequency, 0.3 damping ratio, +-8 cm); off by default, so the
  real car's TF is unchanged
- sim_global.yaml: GNSS covariance for a standalone receiver (1 m / 1.5 m), 5 s of
  antenna averaging at the start
- DESIGN.md: laps driven on the filter at 10 m/s (1 m GNSS: 0.16 m mean, 0.37 m p95)

Co-Authored-By: Claude Opus 5.5 <noreply@anthropic.com>

File: sac_description/urdf/sac.urdf.xacro (robot description, xacro)
@@ -33,4 +33,18 @@
   <xacro:property name="com_x" value="${-wheel_base / 2 + 0.4 * wheel_base}" />
   <xacro:property name="com_z" value="0.55" />
+  <!-- Suspension (not measured): each wheel on a vertical spring and damper. Off by default,
+       so the model is rigid, which is all TF needs on the real car; the simulation turns it
+       on (suspension:=true) so the car does not bounce off bumps and crests.
+       Springs from the corner loads at a 1.4 Hz ride frequency (a usual passenger car value),
+       0.3 damping ratio; travel +-8 cm. -->
+  <xacro:arg name="suspension" default="false" />
+  <xacro:property name="suspension" value="$(arg suspension)" />
+  <xacro:property name="suspension_travel" value="0.08" />        <!-- [m] each way -->
+  <xacro:property name="suspension_frequency" value="1.4" />      <!-- [Hz] -->
+  <xacro:property name="suspension_damping_ratio" value="0.3" />
+  <xacro:property name="suspension_mass" value="5.0" />           <!-- hub and arm, per corner [kg] -->
+  <!-- Sprung mass on each corner, from the axle loads (40/60, see com_x) -->
+  <xacro:property name="front_corner_mass" value="${body_mass * 0.4 / 2}" />
+  <xacro:property name="rear_corner_mass" value="${body_mass * 0.6 / 2}" />
   <xacro:property name="max_speed" value="20.0" />        <!-- [m/s] forward -->
   <xacro:property name="max_reverse_speed" value="5.0" />
@@ -132,10 +146,37 @@
     </link>
   </xacro:macro>
+  <!-- With the suspension, a corner's wheel (or a front wheel's steering) hangs on
+       <corner>_suspension_link, which slides up and down on <corner>_suspension_joint
+       (prismatic, positive = compression); without it, on the chassis. The spring itself is
+       Gazebo's (gazebo_environment), from sac_description's values. -->
+  <xacro:macro name="corner" params="corner x y sprung_mass">
+    <xacro:if value="${suspension}">
+      <xacro:property name="stiffness" value="${sprung_mass * (2 * pi * suspension_frequency) ** 2}" />
+      <link name="${corner}_suspension_link">
+        <xacro:inertial_cuboid mass="${suspension_mass}" x="0.1" y="0.1" z="0.1" />
+      </link>
+      <joint name="${corner}_suspension_joint" type="prismatic">
+        <parent link="link_chassis" />
+        <child link="${corner}_suspension_link" />
+        <origin xyz="${x} ${y} ${wheel_radius}" rpy="0 0 0" />
+        <axis xyz="0 0 1" />
+        <limit effort="100000" velocity="10" lower="${-suspension_travel}" upper="${suspension_travel}" />
+        <dynamics damping="${2 * suspension_damping_ratio * sqrt(stiffness * sprung_mass)}" />
+      </joint>
+    </xacro:if>
+  </xacro:macro>
   <xacro:macro name="rear_wheel" params="side y">
+    <xacro:corner corner="rear_${side}" x="${-wheel_base / 2}" y="${y}" sprung_mass="${rear_corner_mass}" />
     <xacro:wheel_link name="rear_${side}_wheel" />
     <joint name="rear_${side}_wheel_joint" type="continuous">
-      <parent link="link_chassis" />
+      <xacro:if value="${suspension}">
+        <parent link="rear_${side}_suspension_link" />
+        <origin xyz="0 0 0" rpy="${-pi/2} 0 0" />
+      </xacro:if>
+      <xacro:unless value="${suspension}">
+        <parent link="link_chassis" />
+        <origin xyz="${-wheel_base / 2} ${y} ${wheel_radius}" rpy="${-pi/2} 0 0" />
+      </xacro:unless>
       <child link="rear_${side}_wheel" />
-      <origin xyz="${-wheel_base / 2} ${y} ${wheel_radius}" rpy="${-pi/2} 0 0" />
       <axis xyz="0 0 1" />
       <limit effort="1000" velocity="${max_wheel_speed}" />
@@ -143,4 +184,5 @@
   </xacro:macro>
   <xacro:macro name="front_wheel" params="side y">
+    <xacro:corner corner="front_${side}" x="${wheel_base / 2}" y="${y}" sprung_mass="${front_corner_mass}" />
     <!-- 1 kg: a much lighter link between two joints makes the physics unsteady -->
     <link name="front_${side}_wheel_steering_link">
@@ -149,7 +191,13 @@
     <!-- Same frame as the wheel joint, so the steering axis is its -y (the car's up) -->
     <joint name="front_${side}_wheel_steering_joint" type="revolute">
-      <parent link="link_chassis" />
+      <xacro:if value="${suspension}">
+        <parent link="front_${side}_suspension_link" />
+        <origin xyz="0 0 0" rpy="${-pi/2} 0 0" />
+      </xacro:if>
+      <xacro:unless value="${suspension}">
+        <parent link="link_chassis" />
+        <origin xyz="${wheel_base / 2} ${y} ${wheel_radius}" rpy="${-pi/2} 0 0" />
+      </xacro:unless>
       <child link="front_${side}_wheel_steering_link" />
-      <origin xyz="${wheel_base / 2} ${y} ${wheel_radius}" rpy="${-pi/2} 0 0" />
       <axis xyz="0 -1 0" />
       <limit effort="1000" velocity="10" lower="${-steering_limit}" upper="${steering_limit}" />

Commit message: feat: dynamic bicycle motion model; springs carry the whole car
- dynamic_bicycle: bicycle with tyre slip (linear tyres), backward Euler (stable at
  low speed), blended into the kinematic model below 2 m/s; overlay
  config/models/dynamic_bicycle.yaml. 40 % lower yaw error than constant_acceleration
  on a replayed wet lap, but less robust when driving on it, so not the default yet
  (DESIGN.md)
- nonholonomic adapter can be disabled (enabled: false), for models that predict slip
- sac_description: car_mass; the suspension's corner loads are the whole car's, so
  the car stands at the description's height (2-6 mm off instead of 15-19 mm)
- 3 more unit tests (16)

Co-Authored-By: Claude Opus 5.5 <noreply@anthropic.com>

File: sac_description/urdf/sac.urdf.xacro (robot description, xacro)
@@ -44,7 +44,10 @@
   <xacro:property name="suspension_damping_ratio" value="0.3" />
   <xacro:property name="suspension_mass" value="5.0" />           <!-- hub and arm, per corner [kg] -->
-  <!-- Sprung mass on each corner, from the axle loads (40/60, see com_x) -->
-  <xacro:property name="front_corner_mass" value="${body_mass * 0.4 / 2}" />
-  <xacro:property name="rear_corner_mass" value="${body_mass * 0.6 / 2}" />
+  <!-- The whole car: body, wheels, suspension and steering links, roof rack (8 kg) -->
+  <xacro:property name="car_mass" value="${body_mass + 4 * wheel_mass + 4 * suspension_mass + 2 * 1.0 + 8.0}" />
+  <!-- Load on each spring at rest, from the axle loads (40/60, see com_x). The springs carry
+       the whole car in the simulation, so the ride height stays the description's. -->
+  <xacro:property name="front_corner_mass" value="${car_mass * 0.4 / 2}" />
+  <xacro:property name="rear_corner_mass" value="${car_mass * 0.6 / 2}" />
   <xacro:property name="max_speed" value="20.0" />        <!-- [m/s] forward -->
   <xacro:property name="max_reverse_speed" value="5.0" />

Commit message: feat: sac_perception, the local occupancy grid from any number of sensors
Sources per message type (pointcloud, laser_scan, occupancy_grid) set in YAML,
a filter chain per point cloud as plugins (crop_box, voxel, ground_height,
ground_patchwork after Patchwork++, height_band), a rolling grid in odom with
a layer per source, a shared ground map, and a 2D lidar on the car's front.

Co-Authored-By: Claude Opus 5.5 <noreply@anthropic.com>

File: sac_description/urdf/sac.urdf.xacro (robot description, xacro)
@@ -87,4 +87,6 @@
   <xacro:property name="front_imu_xyz" value="${wheel_base / 2} 0 0.5" />
   <xacro:property name="back_imu_xyz" value="${-wheel_base / 2} 0 0.5" />
+  <!-- 2D lidar on the front bumper, level (not measured) -->
+  <xacro:property name="front_lidar_xyz" value="${body_length / 2 + 0.05} 0 0.45" />
   <!-- ============================== Body ============================== -->
   <link name="base_footprint" />
@@ -246,3 +248,6 @@
     <origin xyz="${lidar_xyz}" rpy="0 0 0" />
   </xacro:vlp16>
+  <xacro:lidar_2d name="front_lidar" parent_link="link_chassis">
+    <origin xyz="${front_lidar_xyz}" rpy="0 0 0" />
+  </xacro:lidar_2d>
 </robot>

File: sac_description/urdf/sensors.urdf.xacro (robot description, xacro)
@@ -48,4 +48,25 @@
                     <mesh filename="package://sac_description/meshes/velodyne-vlp16.stl" scale="0.001 0.001 0.001" />
                 </geometry>
+            </visual>
+        </link>
+    </xacro:macro>
+    <!-- ============================== 2D lidar ============================== -->
+    <!-- A generic planar scanner (model not chosen yet); frame <name>_frame at the scan
+         plane's centre, x forward -->
+    <xacro:macro name="lidar_2d" params="name parent_link *origin">
+        <joint name="${name}_joint" type="fixed">
+            <parent link="${parent_link}" />
+            <child link="${name}_frame" />
+            <xacro:insert_block name="origin" />
+        </joint>
+        <link name="${name}_frame">
+            <xacro:inertial_dummy />
+            <visual>
+                <geometry>
+                    <cylinder radius="0.04" length="0.07" />
+                </geometry>
+                <material name="dark_grey">
+                    <color rgba="0.2 0.2 0.2 1.0" />
+                </material>
             </visual>
         </link>
